Commit message: Initial commit - Working warehouse robot with autonomous pallet mission

File: urdf/robot.urdf.xacro (robot description, xacro)
@@ -2,6 +2,7 @@
 <robot name="tracked_robot" xmlns:xacro="http://www.ros.org/wiki/xacro">
   <material name="Orange"><color rgba="1.0 0.45 0.0 1.0"/></material>
-  <material name="Black"><color rgba="0.08 0.08 0.08 1.0"/></material>
-  <material name="Blue"><color rgba="0.1 0.35 0.9 1.0"/></material>
+  <material name="Black"><color rgba="0.1 0.1 0.1 1.0"/></material>
+  <material name="Steel"><color rgba="0.75 0.75 0.8 1.0"/></material>
+  <material name="Rubber"><color rgba="0.2 0.2 0.2 1.0"/></material>
   <link name="base_footprint"/>
   <joint name="base_joint" type="fixed">
@@ -10,44 +11,51 @@
     <origin xyz="0 0 0" rpy="0 0 0"/>
   </joint>
+  <!-- ================= ОСНОВНОЙ КОРПУС ================= -->
+  <!-- Размеры по ТЗ: Длина 492 мм, Ширина 225 мм, Высота шасси 93 мм (с подушкой 95 мм) -->
   <link name="base_link">
+    <!-- Визуальный корпус -->
     <visual>
-      <origin xyz="0 0 0.0475"/>
-      <geometry><box size="0.30 0.12 0.055"/></geometry>
+      <origin xyz="0 0 0.0465"/>
+      <geometry><box size="0.492 0.145 0.073"/></geometry>
       <material name="Orange"/>
     </visual>
+    <!-- Левая гусеничная балка (высота 74 мм) -->
     <visual>
-      <origin xyz="0 0.08 0.03"/>
-      <geometry><box size="0.30 0.04 0.06"/></geometry>
+      <origin xyz="0 0.0925 0.037"/>
+      <geometry><box size="0.492 0.04 0.074"/></geometry>
       <material name="Black"/>
     </visual>
+    <!-- Правая гусеничная балка (высота 74 мм) -->
     <visual>
-      <origin xyz="0 -0.08 0.03"/>
-      <geometry><box size="0.30 0.04 0.06"/></geometry>
+      <origin xyz="0 -0.0925 0.037"/>
+      <geometry><box size="0.492 0.04 0.074"/></geometry>
       <material name="Black"/>
     </visual>
+    <!-- Коллизия корпуса: ширина 216 мм для гарантированного отсутствия заклинивания в проёме 227 мм -->
     <collision>
-      <origin xyz="0 0 0.0475"/>
-      <geometry><box size="0.30 0.12 0.055"/></geometry>
+      <origin xyz="0 0 0.0465"/>
+      <geometry><box size="0.488 0.216 0.073"/></geometry>
     </collision>
     <inertial>
       <origin xyz="0 0 0.045"/>
-      <mass value="15.0"/>
-      <inertia ixx="0.0218" ixy="0" ixz="0" iyy="0.116" iyz="0" izz="0.1305"/>
+      <mass value="25.0"/>
+      <inertia ixx="0.15" ixy="0" ixz="0" iyy="0.55" iyz="0" izz="0.65"/>
     </inertial>
   </link>
+  <!-- Скользящие борта шасси (тефлон, чтобы не залипать на деревянных шашках поддона) -->
+  <gazebo reference="base_link">
+    <mu1>0.05</mu1>
+    <mu2>0.05</mu2>
+  </gazebo>
+  <!-- ================= ПРИВОДНЫЕ КОЛЕСА (СКРЫТЫ В ГУСЕНИЦАХ) ================= -->
   <xacro:macro name="track_wheel" params="name x y">
     <link name="${name}_link">
-      <visual>
-        <origin rpy="${pi/2} 0 0"/>
-        <geometry><cylinder radius="0.031" length="0.042"/></geometry>
-        <material name="Black"/>
-      </visual>
       <collision>
         <origin rpy="${pi/2} 0 0"/>
-        <geometry><cylinder radius="0.03" length="0.04"/></geometry>
+        <geometry><cylinder radius="0.037" length="0.038"/></geometry>
       </collision>
       <inertial>
-        <mass value="0.3"/>
-        <inertia ixx="0.0001075" ixy="0" ixz="0" iyy="0.000135" iyz="0" izz="0.0001075"/>
+        <mass value="1.0"/>
+        <inertia ixx="0.001" ixy="0" ixz="0" iyy="0.001" iyz="0" izz="0.001"/>
       </inertial>
     </link>
@@ -55,27 +63,31 @@
       <parent link="base_link"/>
       <child link="${name}_link"/>
-      <origin xyz="${x} ${y} 0.03"/>
+      <origin xyz="${x} ${y} 0.037"/>
       <axis xyz="0 1 0"/>
     </joint>
     <gazebo reference="${name}_link">
-      <mu1>1.0</mu1>
-      <mu2>1.0</mu2>
+      <mu1>1.8</mu1>
+      <mu2>1.8</mu2>
     </gazebo>
   </xacro:macro>
-  <xacro:track_wheel name="wheel_fl" x="0.11" y="0.08"/>
-  <xacro:track_wheel name="wheel_rl" x="-0.11" y="0.08"/>
-  <xacro:track_wheel name="wheel_fr" x="0.11" y="-0.08"/>
-  <xacro:track_wheel name="wheel_rr" x="-0.11" y="-0.08"/>
+  <xacro:track_wheel name="wheel_fl" x="0.18" y="0.0925"/>
+  <xacro:track_wheel name="wheel_rl" x="-0.18" y="0.0925"/>
+  <xacro:track_wheel name="wheel_fr" x="0.18" y="-0.0925"/>
+  <xacro:track_wheel name="wheel_rr" x="-0.18" y="-0.0925"/>
+  <!-- ================= ПНЕВМОПОДЪЕМНИК ================= -->
+  <!-- Высота в сложенном виде: 2 мм (с 93 мм до 95 мм). Ход: 45 мм -->
   <link name="lift_plate_link">
     <visual>
-      <geometry><box size="0.28 0.19 0.02"/></geometry>
-      <material name="Blue"/>
+      <origin xyz="0 0 0.001"/>
+      <geometry><box size="0.470 0.210 0.002"/></geometry>
+      <material name="Rubber"/>
     </visual>
     <collision>
-      <geometry><box size="0.28 0.19 0.02"/></geometry>
+      <origin xyz="0 0 0.001"/>
+      <geometry><box size="0.470 0.210 0.002"/></geometry>
     </collision>
     <inertial>
-      <mass value="2.0"/>
-      <inertia ixx="0.00608" ixy="0" ixz="0" iyy="0.01313" iyz="0" izz="0.01908"/>
+      <mass value="3.0"/>
+      <inertia ixx="0.01" ixy="0" ixz="0" iyy="0.05" iyz="0" izz="0.06"/>
     </inertial>
   </link>
@@ -83,24 +95,17 @@
     <parent link="base_link"/>
     <child link="lift_plate_link"/>
-    <origin xyz="0 0 0.085"/>
+    <!-- Установлен ровно на отметке 93 мм от пола: 93 + 2 = 95 мм общая высота -->
+    <origin xyz="0 0 0.093"/>
     <axis xyz="0 0 1"/>
-    <limit lower="0.0" upper="0.05" effort="3000" velocity="0.03"/>
-    <dynamics damping="50.0" friction="10.0"/>
+    <!-- Ход от 0 до 45 мм с усилием пневматики 4000 Н (грузоподъемность > 300 кг) -->
+    <limit lower="0.0" upper="0.045" effort="4000" velocity="0.04"/>
+    <dynamics damping="80.0" friction="5.0"/>
   </joint>
-  <link name="laser_link">
-    <visual>
-      <geometry><cylinder radius="0.01" length="0.02"/></geometry>
-      <material name="Black"/>
-    </visual>
-    <inertial>
-      <mass value="0.05"/>
-      <inertia ixx="0.00001" ixy="0" ixz="0" iyy="0.00001" iyz="0" izz="0.00001"/>
-    </inertial>
-  </link>
-  <joint name="laser_joint" type="fixed">
-    <parent link="base_link"/>
-    <child link="laser_link"/>
-    <origin xyz="0.145 0 0.05"/>
-  </joint>
+  <!-- Высокое трение площадки, чтобы поддон не соскальзывал при подъёме -->
+  <gazebo reference="lift_plate_link">
+    <mu1>2.0</mu1>
+    <mu2>2.0</mu2>
+  </gazebo>
+  <!-- ================= ПЛАГИНЫ ДЛЯ GAZEBO HARMONIC ================= -->
   <gazebo>
     <plugin filename="gz-sim-diff-drive-system" name="gz::sim::systems::DiffDrive">
@@ -109,25 +114,26 @@
       <right_joint>wheel_fr_joint</right_joint>
       <right_joint>wheel_rr_joint</right_joint>
-      <wheel_separation>0.16</wheel_separation>
-      <wheel_radius>0.03</wheel_radius>
+      <wheel_separation>0.185</wheel_separation>
+      <wheel_radius>0.037</wheel_radius>
       <odom_publish_frequency>50</odom_publish_frequency>
-      <max_linear_acceleration>0.5</max_linear_acceleration>
-      <max_angular_acceleration>1.5</max_angular_acceleration>
-      <max_velocity>0.5</max_velocity>
+      <max_linear_acceleration>1.0</max_linear_acceleration>
+      <min_linear_acceleration>-1.0</min_linear_acceleration>
+      <max_angular_acceleration>2.0</max_angular_acceleration>
+      <min_angular_acceleration>-2.0</min_angular_acceleration>
+      <max_velocity>0.6</max_velocity>
       <topic>/cmd_vel</topic>
       <odom_topic>/odom</odom_topic>
-      <odom_frame>odom</odom_frame>
-      <robot_base_frame>base_footprint</robot_base_frame>
+      <tf_topic>/tf</tf_topic>
+      <frame_id>odom</frame_id>
+      <child_frame_id>base_footprint</child_frame_id>
     </plugin>
     <plugin filename="gz-sim-joint-position-controller-system" name="gz::sim::systems::JointPositionController">
       <joint_name>lift_joint</joint_name>
       <topic>/lift_cmd</topic>
-      <p_gain>5000.0</p_gain>
-      <i_gain>100.0</i_gain>
-      <d_gain>500.0</d_gain>
-      <i_max>1000.0</i_max>
-      <i_min>-1000.0</i_min>
-      <cmd_max>3000.0</cmd_max>
-      <cmd_min>-3000.0</cmd_min>
+      <p_gain>10000.0</p_gain>
+      <i_gain>500.0</i_gain>
+      <d_gain>800.0</d_gain>
+      <cmd_max>4000.0</cmd_max>
+      <cmd_min>-1000.0</cmd_min>
     </plugin>
     <plugin filename="gz-sim-joint-state-publisher-system" name="gz::sim::systems::JointStatePublisher">
